Commit message: change demo05 file

File: demo05_ws/src/urdf02_gazebo/urdf/demo05_car_base.urdf.xacro (robot description, xacro)
@@ -20,5 +20,5 @@
             <origin xyz="0 0 0" rpy="0 0 0" />
             <material name="baselink_color">
-                <color rgba="1.0 0.5 0.2 0.5" />
+                <color rgba="0.2 0.2 0.2 0.5" />
             </material>
         </visual>
@@ -32,5 +32,5 @@
     </link>
     <gazebo reference="base_link">
-        <material>Gazebo/Yellow</material>
+        <material>Gazebo/Grey</material>
     </gazebo>
     <joint name="link2footprint" type="fixed">
@@ -64,5 +64,5 @@
         </link>
         <gazebo reference="${wheel_name}_wheel">
-            <material>Gazebo/Red</material>
+            <material>Gazebo/Grey</material>
         </gazebo>
         <joint name="${wheel_name}2link" type="continuous">
@@ -99,5 +99,5 @@
         </link>
         <gazebo reference="${small_wheel_name}_wheel">
-            <material>Gazebo/Red</material>
+            <material>Gazebo/Grey</material>
         </gazebo>
         <joint name="${small_wheel_name}2link" type="continuous">

File: demo05_ws/src/urdf02_gazebo/urdf/demo06_car_camera.urdf.xacro (robot description, xacro)
@@ -26,5 +26,5 @@
     </link>
     <gazebo reference="camera">
-        <material>Gazebo/Blue</material>
+        <material>Gazebo/Grey</material>
     </gazebo>
     <joint name="camera2base" type="fixed">

File: demo05_ws/src/urdf02_gazebo/urdf/demo07_car_laser.urdf.xacro (robot description, xacro)
@@ -13,5 +13,5 @@
             <origin xyz="0.0 0.0 0.0" rpy="0.0 0.0 0.0" />
             <material name="red">
-                <color rgba="0.8 0.5 0.0 0.5" />
+                <color rgba="0.1 0.1 0.1 0.5" />
             </material>
         </visual>
